File: PCB/Macropad.kicad_pcb (KiCad board)
At the start: 2 copper layers, 80.2 x 42.4 mm, 7 parts, among them SW1 SW_Push, SW2 SW_Push, SW3 SW_Push, SW4 SW_Push, U1 XIAO-RP2040-DIP

Commit message: Update PCB layout and schematic
Parts:
- removed D2: SK6812, LED_SMD:LED_SK6812MINI_PLCC4_3.5x3.5mm_P1.75mm
- added D3: SK6812MINI-E, Hackclub Footprints:MX_SK6812MINI-E_REV, F.Cu at (123.0, 104.1)
- D1: value SK6812 -> SK6812MINI-E; footprint LED_SMD:LED_SK6812MINI_PLCC4_3.5x3.5mm_P1.75mm -> Hackclub Footprints:MX_SK6812MINI-E_REV
- moved D1 12.6 mm to (132.2, 114.3), turned to 180 degrees
Connections:
- D1 pad 1: GND -> +5V
- D1 pad 2: Net-(D1-DIN) (its old number) -> unconnected-(D1-DOUT-Pad2)
- D1 pad 3: +5V -> GND
- U1 pad 5: Net-(D1-DIN) (its old number) -> Net-(D3-DIN)
Routing:
- net Net-(D3-DIN): track 0.00 -> 17.8 mm
- net Net-(D1-DIN) (its old number): track 16.4 -> 0.00 mm
- net +5V: track 12.6 -> 4.65 mm
- net GND: track 91.8 -> 97.1 mm
- net Net-(D1-DIN): track 9.23 -> 11.6 mm

Commit message: Update PCB layout and schematic
Connections:
- U1 pad 13: unconnected-(U1-GND-Pad13) -> GND
- U1 pad 14: unconnected-(U1-VBUS-Pad14) -> +5V
Routing:
- net GND: track 97.1 -> 168.3 mm
- net +5V: track 4.65 -> 55.3 mm
Changed lines of the file:
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@@
 	(net 8 "unconnected-(U1-GPIO27{slash}ADC1{slash}A1-Pad2)")
 	(net 9 "unconnected-(U1-3V3-Pad12)")
-	(net 10 "unconnected-(U1-VBUS-Pad14)")
-	(net 11 "unconnected-(U1-GPIO29{slash}ADC3{slash}A3-Pad4)")
-	(net 12 "unconnected-(U1-GND-Pad13)")
-	(net 13 "unconnected-(U1-GPIO26{slash}ADC0{slash}A0-Pad1)")
-	(net 14 "unconnected-(U1-GPIO0{slash}TX-Pad7)")
-	(net 15 "unconnected-(U1-GPIO28{slash}ADC2{slash}A2-Pad3)")
-	(net 16 "unconnected-(U1-GPIO7{slash}SCL-Pad6)")
-	(net 17 "unconnected-(D1-DOUT-Pad2)")
-	(net 18 "Net-(D3-DIN)")
+	(net 10 "unconnected-(U1-GPIO29{slash}ADC3{slash}A3-Pad4)")
+	(net 11 "unconnected-(U1-GPIO26{slash}ADC0{slash}A0-Pad1)")
+	(net 12 "unconnected-(U1-GPIO0{slash}TX-Pad7)")
+	(net 13 "unconnected-(U1-GPIO28{slash}ADC2{slash}A2-Pad3)")
+	(net 14 "unconnected-(U1-GPIO7{slash}SCL-Pad6)")
+	(net 15 "unconnected-(D1-DOUT-Pad2)")
+	(net 16 "Net-(D3-DIN)")
 	(footprint "OPL library:XIAO-RP2040-DIP"
 		(layer "F.Cu")
@@
 			(layers "F.Cu" "F.Mask")
 			(roundrect_rratio 0.1)
-			(net 13 "unconnected-(U1-GPIO26{slash}ADC0{slash}A0-Pad1)")
+			(net 11 "unconnected-(U1-GPIO26{slash}ADC0{slash}A0-Pad1)")
 			(pinfunction "GPIO26/ADC0/A0")
 			(pintype "passive")
@@
 			(layers "*.Cu" "*.Mask")
 			(remove_unused_layers no)
-			(net 13 "unconnected-(U1-GPIO26{slash}ADC0{slash}A0-Pad1)")
+			(net 11 "unconnected-(U1-GPIO26{slash}ADC0{slash}A0-Pad1)")
 			(pinfunction "GPIO26/ADC0/A0")
 			(pintype "passive")
@@
 			(layers "F.Cu" "F.Mask")
 			(roundrect_rratio 0.1)
-			(net 15 "unconnected-(U1-GPIO28{slash}ADC2{slash}A2-Pad3)")
+			(net 13 "unconnected-(U1-GPIO28{slash}ADC2{slash}A2-Pad3)")
 			(pinfunction "GPIO28/ADC2/A2")
 			(pintype "passive")
@@
 			(layers "*.Cu" "*.Mask")
 			(remove_unused_layers no)
-			(net 15 "unconnected-(U1-GPIO28{slash}ADC2{slash}A2-Pad3)")
+			(net 13 "unconnected-(U1-GPIO28{slash}ADC2{slash}A2-Pad3)")
 			(pinfunction "GPIO28/ADC2/A2")
 			(pintype "passive")
@@
 			(layers "F.Cu" "F.Mask")
 			(roundrect_rratio 0.1)
-			(net 11 "unconnected-(U1-GPIO29{slash}ADC3{slash}A3-Pad4)")
+			(net 10 "unconnected-(U1-GPIO29{slash}ADC3{slash}A3-Pad4)")
 			(pinfunction "GPIO29/ADC3/A3")
 			(pintype "passive")
@@
 			(layers "*.Cu" "*.Mask")
 			(remove_unused_layers no)
-			(net 11 "unconnected-(U1-GPIO29{slash}ADC3{slash}A3-Pad4)")
+			(net 10 "unconnected-(U1-GPIO29{slash}ADC3{slash}A3-Pad4)")
 			(pinfunction "GPIO29/ADC3/A3")
 			(pintype "passive")
@@
 			(layers "F.Cu" "F.Mask")
 			(roundrect_rratio 0.1)
-			(net 18 "Net-(D3-DIN)")
+			(net 16 "Net-(D3-DIN)")
 			(pinfunction "GPIO6/SDA")
 			(pintype "passive")
@@
 			(layers "*.Cu" "*.Mask")
 			(remove_unused_layers no)
-			(net 18 "Net-(D3-DIN)")
+			(net 16 "Net-(D3-DIN)")
 			(pinfunction "GPIO6/SDA")
 			(pintype "passive")
@@
 			(layers "F.Cu" "F.Mask")
 			(roundrect_rratio 0.1)
-			(net 16 "unconnected-(U1-GPIO7{slash}SCL-Pad6)")
+			(net 14 "unconnected-(U1-GPIO7{slash}SCL-Pad6)")
 			(pinfunction "GPIO7/SCL")
 			(pintype "passive")
@@
 			(layers "*.Cu" "*.Mask")
 			(remove_unused_layers no)
-			(net 16 "unconnected-(U1-GPIO7{slash}SCL-Pad6)")
+			(net 14 "unconnected-(U1-GPIO7{slash}SCL-Pad6)")
 			(pinfunction "GPIO7/SCL")
 			(pintype "passive")
@@
 			(layers "F.Cu" "F.Mask")
 			(roundrect_rratio 0.1)
-			(net 14 "unconnected-(U1-GPIO0{slash}TX-Pad7)")
+			(net 12 "unconnected-(U1-GPIO0{slash}TX-Pad7)")
 			(pinfunction "GPIO0/TX")
 			(pintype "passive")
@@
 			(layers "*.Cu" "*.Mask")
 			(remove_unused_layers no)
-			(net 14 "unconnected-(U1-GPIO0{slash}TX-Pad7)")
+			(net 12 "unconnected-(U1-GPIO0{slash}TX-Pad7)")
 			(pinfunction "GPIO0/TX")
 			(pintype "passive")
@@
 			(layers "*.Cu" "*.Mask")
 			(remove_unused_layers no)
-			(net 12 "unconnected-(U1-GND-Pad13)")
+			(net 2 "GND")
 			(pinfunction "GND")
 			(pintype "passive")
@@
 			(layers "F.Cu" "F.Mask")
 			(roundrect_rratio 0.1)
-			(net 12 "unconnected-(U1-GND-Pad13)")
+			(net 2 "GND")
 			(pinfunction "GND")
 			(pintype "passive")
@@
 			(layers "*.Cu" "*.Mask")
 			(remove_unused_layers no)
-			(net 10 "unconnected-(U1-VBUS-Pad14)")
+			(net 3 "+5V")
 			(pinfunction "VBUS")
 			(pintype "passive")
@@
 			(layers "F.Cu" "F.Mask")
 			(roundrect_rratio 0.1)
-			(net 10 "unconnected-(U1-VBUS-Pad14)")
+			(net 3 "+5V")
 			(pinfunction "VBUS")
 			(pintype "passive")
@@
 			(layers "B.Cu" "B.Mask" "B.Paste")
 			(roundrect_rratio 0.1)
-			(net 17 "unconnected-(D1-DOUT-Pad2)")
+			(net 15 "unconnected-(D1-DOUT-Pad2)")
 			(pinfunction "DOUT")
 			(pintype "output")
@@
 			(layers "B.Cu" "B.Mask" "B.Paste")
 			(roundrect_rratio 0.1)
-			(net 18 "Net-(D3-DIN)")
+			(net 16 "Net-(D3-DIN)")
 			(pinfunction "DIN")
 			(pintype "input")
@@
 	)
 	(segment
+		(start 186.434375 96.737275)
+		(end 175.0961 85.399)
+		(width 0.2)
+		(layer "B.Cu")
+		(net 2)
+	)
+	(segment
 		(start 120.35 108.44)
 		(end 120.35 107.21)
@@
 	)
 	(segment
+		(start 151.421 85.399)
+		(end 147.539624 89.280376)
+		(width 0.2)
+		(layer "B.Cu")
+		(net 2)
+	)
+	(segment
+		(start 136.15 109.44)
+		(end 135.6 109.99)
+		(width 0.2)
+		(layer "B.Cu")
+		(net 2)
+	)
+	(segment
+		(start 121.57 105.99)
+		(end 136.15 105.99)
+		(width 0.2)
+		(layer "B.Cu")
+		(net 2)
+	)
+	(segment
+		(start 136.15 105.99)
+		(end 136.15 109.44)
+		(width 0.2)
+		(layer "B.Cu")
+		(net 2)
+	)
+	(segment
 		(start 120.35 107.21)
-		(end 122.05 105.51)
+		(end 121.57 105.99)
 		(width 0.2)
 		(layer "B.Cu")
@@
 	)
 	(segment
-		(start 122.05 105.51)
-		(end 136.15 105.51)
+		(start 141.566745 113.60806)
+		(end 143.440875 113.60806)
 		(width 0.2)
 		(layer "B.Cu")
@@
 	)
 	(segment
-		(start 141.566745 113.60806)
-		(end 143.440875 113.60806)
-		(width 0.2)
-		(layer "B.Cu")
-		(net 2)
-	)
-	(segment
 		(start 137.948685 109.99)
 		(end 141.566745 113.60806)
@@
 	)
 	(segment
+		(start 175.0961 85.399)
+		(end 151.421 85.399)
+		(width 0.2)
+		(layer "B.Cu")
+		(net 2)
+	)
+	(segment
+		(start 147.539624 89.280376)
+		(end 133.661875 89.280376)
+		(width 0.2)
+		(layer "B.Cu")
+		(net 2)
+	)
+	(segment
 		(start 143.440875 113.60806)
 		(end 147.547059 109.501876)
@@
 	)
 	(segment
-		(start 136.15 105.51)
-		(end 136.15 109.44)
+		(start 186.434375 109.501876)
+		(end 186.434375 96.737275)
 		(width 0.2)
 		(layer "B.Cu")
@@
 	)
 	(segment
-		(start 136.15 109.44)
-		(end 135.6 109.99)
-		(width 0.2)
-		(layer "B.Cu")
-		(net 2)
+		(start 132.598875 87.803376)
+		(end 133.661875 86.740376)
+		(width 0.2)
+		(layer "B.Cu")
+		(net 3)
 	)
 	(segment
@@
 	)
 	(segment
+		(start 117.981565 87.803376)
+		(end 132.598875 87.803376)
+		(width 0.2)
+		(layer "B.Cu")
+		(net 3)
+	)
+	(segment
+		(start 120.55 111.67)
+		(end 119.531 110.651)
+		(width 0.2)
+		(layer "B.Cu")
+		(net 3)
+	)
+	(segment
+		(start 126.27 111.67)
+		(end 120.55 111.67)
+		(width 0.2)
+		(layer "B.Cu")
+		(net 3)
+	)
+	(segment
+		(start 119.249 110.369)
+		(end 115.749 106.869)
+		(width 0.2)
+		(layer "B.Cu")
+		(net 3)
+	)
+	(segment
+		(start 115.749 90.035941)
+		(end 117.981565 87.803376)
+		(width 0.2)
+		(layer "B.Cu")
+		(net 3)
+	)
+	(segment
+		(start 115.749 106.869)
+		(end 115.749 90.035941)
+		(width 0.2)
+		(layer "B.Cu")
+		(net 3)
+	)
+	(segment
+		(start 119.471086 110.651)
+		(end 119.249 110.428914)
+		(width 0.2)
+		(layer "B.Cu")
+		(net 3)
+	)
+	(segment
+		(start 125.55 109.94)
+		(end 126.27 110.66)
+		(width 0.2)
+		(layer "B.Cu")
+		(net 3)
+	)
+	(segment
+		(start 119.249 110.428914)
+		(end 119.249 110.369)
+		(width 0.2)
+		(layer "B.Cu")
+		(net 3)
+	)
+	(segment
 		(start 126.35 109.94)
 		(end 127.8 108.49)
@@
 	)
 	(segment
+		(start 126.27 110.66)
+		(end 126.27 111.67)
+		(width 0.2)
+		(layer "B.Cu")
+		(net 3)
+	)
+	(segment
+		(start 119.531 110.651)
+		(end 119.471086 110.651)
+		(width 0.2)
+		(layer "B.Cu")
+		(net 3)
+	)
+	(segment
 		(start 127.8 108.49)
 		(end 129.6 108.49)
@@
 	)
 	(segment
+		(start 138.062251 89.96)
+		(end 133.661875 94.360376)
+		(width 0.2)
+		(layer "B.Cu")
+		(net 7)
+	)
+	(segment
+		(start 174.93 85.8)
+		(end 152.03 85.8)
+		(width 0.2)
+		(layer "B.Cu")
+		(net 7)
+	)
+	(segment
+		(start 147.87 89.96)
+		(end 138.062251 89.96)
+		(width 0.2)
+		(layer "B.Cu")
+		(net 7)
+	)
+	(segment
 		(start 180.084375 90.954375)
 		(end 174.93 85.8)
@@
 	)
 	(segment
+		(start 152.03 85.8)
+		(end 147.87 89.96)
+		(width 0.2)
+		(layer "B.Cu")
+		(net 7)
+	)
+	(segment
 		(start 180.084375 112.041876)
 		(end 180.084375 90.954375)
@@
 	)
 	(segment
-		(start 174.93 85.8)
-		(end 152.03 85.8)
-		(width 0.2)
-		(layer "B.Cu")
-		(net 7)
-	)
-	(segment
-		(start 143.469624 94.360376)
-		(end 133.661875 94.360376)
-		(width 0.2)
-		(layer "B.Cu")
-		(net 7)
-	)
-	(segment
-		(start 152.03 85.8)
-		(end 143.469624 94.360376)
-		(width 0.2)
-		(layer "B.Cu")
-		(net 7)
-	)
-	(segment
 		(start 116.329624 96.900376)
 		(end 118.421875 96.900376)
 		(width 0.2)
 		(layer "B.Cu")
-		(net 18)
-	)
-	(segment
-		(start 115.68 106.07)
-		(end 115.68 97.55)
-		(width 0.2)
-		(layer "B.Cu")
-		(net 18)
-	)
-	(segment
-		(start 115.68 97.55)
+		(net 16)
+	)
+	(segment
+		(start 119.55 109.94)
+		(end 116.15 106.54)
+		(width 0.2)
+		(layer "B.Cu")
+		(net 16)
+	)
+	(segment
+		(start 116.15 106.54)
+		(end 116.15 97.08)
+		(width 0.2)
+		(layer "B.Cu")
+		(net 16)
+	)
+	(segment
+		(start 116.15 97.08)
 		(end 116.329624 96.900376)
 		(width 0.2)
 		(layer "B.Cu")
-		(net 18)
+		(net 16)
 	)
 	(segment
@@
 		(width 0.2)
 		(layer "B.Cu")
-		(net 18)
-	)
-	(segment
-		(start 119.55 109.94)
-		(end 115.68 106.07)
-		(width 0.2)
-		(layer "B.Cu")
-		(net 18)
+		(net 16)
 	)
 	(embedded_fonts no)
